File: RFID-mobileV_1_0/_autosave-RFID-mobileV_1_0.kicad_sch (KiCad schematic)
At the start: 52 parts, among them J1 USB_C_Receptacle_USB2.0, Q1 MMBT3904, SW1 SW_Push, U1 XC6206P332MR, U2 E22-400T22S, U3 STM32G030FxP, U4 LM321, U5 TP4054

Commit message: add jlcpcb
Parts:
- C5: value C -> (none); footprint Capacitor_SMD:C_0805_2012Metric -> (none)
Changed lines of the file:
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@@
       (effects (font (size 1.27 1.27)) (justify left))
     )
-    (property "Value" "C" (id 1) (at 161.29 46.3549 0)
-      (effects (font (size 1.27 1.27)) (justify left))
-    )
-    (property "Footprint" "Capacitor_SMD:C_0805_2012Metric" (id 2) (at 158.4452 48.895 0)
+    (property "Value" "" (id 1) (at 161.29 46.3549 0)
+      (effects (font (size 1.27 1.27)) (justify left))
+    )
+    (property "Footprint" "" (id 2) (at 158.4452 48.895 0)
       (effects (font (size 1.27 1.27)) hide)
     )
@@
     )
     (path "/600d1817-b711-4dc4-847d-e60b9198af7b"
-      (reference "C5") (unit 1) (value "C") (footprint "Capacitor_SMD:C_0805_2012Metric")
+      (reference "C5") (unit 1) (value "0.1uF") (footprint "Capacitor_SMD:C_0805_2012Metric")
     )
     (path "/d5f34cdc-c982-4ea2-9952-8b32c1792e7d"
